File: pcb/audio.kicad_sch (KiCad schematic)
At the start: 15 parts, among them CN1 PJ-325C5-G, U7 PCM2704CDBR, Y3 12Mhz

Commit message: added bom to readme, completed project
Parts:
- Y3: LCSC Part # C9006 -> C5280578
Changed lines of the file:
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@@
 			)
 		)
-		(property "LCSC Part #" "C9006"
+		(property "LCSC Part #" "C5280578"
 			(at 260.35 24.13 0)
 			(effects

Commit message: add gerbers
Parts:
- removed CN1: PJ-325C5-G, easyeda2kicad:AUDIO-TH_PJ-325C5-G, symbol easyeda2kicad:PJ-325C5-G
- added U8: PJ-320A-4P DIP, easyeda2kicad:AUDIO-TH_PJ-320A-4P-DIP, symbol easyeda2kicad:PJ-320A-4PDIP
Connections:
- net GND: now also U8.A, U8.B
- net at U7.14 (VOUTL): now also U8.D
- net at U7.15 (VOUTR): now also U8.C
