File: pcb/skibidi-thinkbook-14-hub.kicad_pcb (KiCad board)
At the start: 4 copper layers, 40 x 70 mm, 121 parts, among them CN1 PJ-325C5-G, U1 HC-USB3.0-C26, U2 TUSB8042AIRGCR, U3 RTL8153B-VB-CG, U4 CH334P, U5 AP63203WU-7, U6 CYA0650-4.7UH, U7 PCM2704CDBR, Y1 24Mhz, Y2 25Mhz, Y3 12Mhz

Commit message: add gerbers
Parts:
- removed CN1: PJ-325C5-G, easyeda2kicad:AUDIO-TH_PJ-325C5-G
- added U8: PJ-320A-4P DIP, easyeda2kicad:AUDIO-TH_PJ-320A-4P-DIP, F.Cu at (135.5, 111.2)
Routing:
- net Net-(U7-VOUTL): track 17.2 -> 18.6 mm
- net Net-(U7-VOUTR): track 17.5 -> 16.6 mm
